File: hardware/tap.kicad_pcb (KiCad board)
At the start: 4 copper layers, 80 x 80 mm, 56 parts, among them CON1 USB-MINI-B, P1 H, P10 D, P11 H, P12 HTAP, P13 PTAP, P14 DTAP, P15 D, P16 H, P17 HTAP, P18 PTAP, P19 DTAP, P2 HTAP, P20 D, P21 ICSP, P22 CONN_1, P23 CONN_1, P3 PTAP, P4 DTAP, P5 D, P6 H, P7 HTAP, P8 PTAP, P9 DTAP, U1 G6K-2F-RF, U10 PIC16F1454, U11 74LS595, U12 74LS595, U13 MMA8653FC, U2 G6K-2F-RF, U3 G6K-2F-RF, U4 G6K-2F-RF, U5 G6K-2F-RF, U6 G6K-2F-RF, U7 G6K-2F-RF, U8 G6K-2F-RF, U9 3v3

Commit message: fixing my shit
Parts:
- removed P13, P18: PTAP, 00-9176-002
- removed VAL: REF, bb
- added HOLE: VAL**, HOLE, F.Cu at (166.0, 92.0)
- added HOLE: VAL**, HOLE, F.Cu at (100.0, 153.0)
- added HOLE: VAL**, HOLE, F.Cu at (160.0, 153.0)
- added HOLE: VAL**, HOLE, F.Cu at (130.0, 153.0)
- added HOLE: VAL**, HOLE, F.Cu at (94.0, 92.0)
- added HOLE: VAL**, HOLE, F.Cu at (130.0, 81.0)
- P3, P8: value PTAP -> CONN_1; footprint 00-9176-002 -> 1pin
- moved P22 57.0 mm to (93.0, 154.0)
- moved P23 57.0 mm to (167.0, 154.0)
- moved R6 43.9 mm to (159.0, 86.0), turned to 90 degrees
- moved C8 43.1 mm to (156.0, 83.0), turned to 0 degrees
- moved P8 42.1 mm to (167.0, 98.0)
- moved U13 40.4 mm to (156.0, 86.0), turned to 0 degrees
- moved C4 37.1 mm to (150.0, 83.0), turned to 180 degrees
- moved R5 37.1 mm to (153.0, 86.0), turned to 270 degrees
- moved C9 37.1 mm to (155.0, 89.0), turned to 180 degrees
- moved P21 36.4 mm to (143.5, 80.0)
- moved U9 34.0 mm to (150.0, 86.0), turned to 270 degrees
- moved L1 32.8 mm to (97.8, 96.4)
- moved D2 32.0 mm to (123.9, 80.2), turned to 0 degrees
- moved C5 31.1 mm to (150.0, 89.0), turned to 0 degrees
- moved P3 22.2 mm to (93.0, 98.0)
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Connections:
- P1 pad 1: N-0000051 -> N-0000043
- P1 pad 2: N-0000045 -> N-0000042
- P10 pad 1: N-0000060 -> N-0000055
- P10 pad 2: N-0000052 -> N-0000056
- P11 pad 1: N-0000071 -> N-0000059
- P11 pad 2: N-0000065 -> N-0000058
- P12 pad 1: N-0000066 -> N-0000065
- P12 pad 2: N-0000067 -> N-0000060
- P14 pad 1: N-0000064 -> N-0000061
- P14 pad 2: N-0000069 -> N-0000062
- P15 pad 1: N-0000070 -> N-0000063
- P15 pad 2: N-0000063 -> N-0000064
- P16 pad 1: N-0000081 -> N-0000068
- P16 pad 2: N-0000075 -> N-0000066
- P17 pad 1: N-0000076 -> N-0000073
- P17 pad 2: N-0000077 -> N-0000067
- P19 pad 1: N-0000074 -> N-0000069
- P19 pad 2: N-0000079 -> N-0000070
- P2 pad 1: N-0000047 -> N-0000049
- P2 pad 2: N-0000046 -> N-0000044
- P20 pad 1: N-0000080 -> N-0000071
- P3 pad 1: N-0000048 -> AGND
- P4 pad 1: N-0000044 -> N-0000045
- P4 pad 2: N-0000049 -> N-0000046
- P5 pad 1: N-0000050 -> N-0000047
- P5 pad 2: N-0000042 -> N-0000048
- P6 pad 1: N-0000061 -> N-0000050
- P6 pad 2: N-0000055 -> N-0000051
- P7 pad 1: N-0000056 -> N-0000057
- P7 pad 2: N-0000057 -> N-0000053
- P8 pad 1: N-0000058 -> AGND
- P9 pad 2: N-0000059 -> N-0000052
- U1 pad 2: N-0000046 -> N-0000044
- U1 pad 3: N-0000045 -> N-0000042
- U1 pad 4: N-0000043 -> N-0000048
- U1 pad 5: N-0000048 -> N-0000047
- U1 pad 6: N-0000051 -> N-0000043
- U1 pad 7: N-0000047 -> N-0000049
- U12 pad 1: /1/DC- -> /1/DC+
- U12 pad 15: /1/DC+ -> /1/DC-
- U12 pad 2: /2/DC+ -> /2/DC-
- U12 pad 3: /2/DC- -> /2/DC+
- U12 pad 4: /3/DC+ -> /3/DC-
- U12 pad 5: /3/DC- -> /3/DC+
- U12 pad 6: /4/DC+ -> /4/DC-
- U12 pad 7: /4/DC- -> /4/DC+
- U2 pad 2: N-0000045 -> N-0000047
- U2 pad 3: N-0000042 -> N-0000045
- U2 pad 6: N-0000050 -> N-0000046
- U2 pad 7: N-0000051 -> N-0000048
- U3 pad 2: N-0000057 -> N-0000053
- U3 pad 3: N-0000055 -> N-0000051
- U3 pad 4: N-0000053 -> N-0000056
- U3 pad 5: N-0000058 -> N-0000055
- U3 pad 6: N-0000061 -> N-0000050
- U3 pad 7: N-0000056 -> N-0000057
- U4 pad 3: N-0000052 -> N-0000054
- U4 pad 4: N-0000059 -> N-0000057
- U4 pad 5: N-0000054 -> N-0000053
- U4 pad 6: N-0000060 -> N-0000052
- U4 pad 7: N-0000061 -> N-0000056
- U5 pad 2: N-0000067 -> N-0000060
- U5 pad 3: N-0000065 -> N-0000058
- U5 pad 4: N-0000062 -> N-0000064
- U5 pad 5: N-0000068 -> N-0000063
- U5 pad 6: N-0000071 -> N-0000059
- U5 pad 7: N-0000066 -> N-0000065
- U6 pad 2: N-0000065 -> N-0000063
- U6 pad 3: N-0000063 -> N-0000061
- U6 pad 4: N-0000069 -> N-0000065
- U6 pad 5: N-0000064 -> N-0000060
- U6 pad 6: N-0000070 -> N-0000062
- U6 pad 7: N-0000071 -> N-0000064
- U7 pad 2: N-0000077 -> N-0000067
- U7 pad 3: N-0000075 -> N-0000066
- U7 pad 4: N-0000073 -> N-0000072
- U7 pad 5: N-0000078 -> N-0000071
- U7 pad 6: N-0000081 -> N-0000068
- U7 pad 7: N-0000076 -> N-0000073
- U8 pad 2: N-0000075 -> N-0000071
- U8 pad 3: N-0000072 -> N-0000069
- U8 pad 4: N-0000079 -> N-0000073
- U8 pad 5: N-0000074 -> N-0000067
- U8 pad 6: N-0000080 -> N-0000070
- U8 pad 7: N-0000081 -> N-0000072
Routing:
- net N-0000075: track 106.2 -> 0.00 mm
- net N-0000081: track 106.2 -> 0.00 mm
- net VCC: track 130.6 -> 41.9 mm, vias 2 -> 4
- net N-0000061: track 106.2 -> 28.7 mm, vias 0 -> 2
- net N-0000051: track 106.2 -> 35.4 mm
- net N-0000065: track 106.2 -> 44.4 mm, vias 0 -> 3
- net N-0000080: track 55.6 -> 0.00 mm
- net N-0000055: track 106.2 -> 51.6 mm
- net N-0000071: track 106.2 -> 51.6 mm
- net N-0000078: track 53.9 -> 0.00 mm, vias 3 -> 0
- net N-0000045: track 106.2 -> 61.7 mm, vias 0 -> 2
- net /SDA: track 21.9 -> 61.5 mm, vias 1 -> 3
- net /MCLR: track 10.9 -> 43.8 mm
- net /SCL: track 29.6 -> 59.7 mm, vias 1 -> 3
- net /1/DC+: track 37.8 -> 8.04 mm, vias 2 -> 0
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- added copper zone on Inner2.Cu, net GND
- added copper zone on Inner1.Cu, net VCC
- removed copper zone on B.Cu, net GND
Other:
- outline, holes or cut-outs redrawn
- board text added: "Eric Van Albert Zach Banks"
- board text added: "Universal Tap rev 3"
- board text removed: "PASSIVE TAP"
- board text removed: "Universal Tap rev 1"
